Commit message: connect RealSense to last link via camera mount

File: mul_franka_description/robots/panda_arm.urdf.xacro (robot description, xacro)
@@ -6,4 +6,5 @@
   <xacro:arg name="use_fake_hardware" default="false"/>
   <xacro:arg name="fake_sensor_commands" default="false"/>
+  <xacro:arg name="add_realsense" default="false"/>
   <xacro:include filename="$(find franka_description)/robots/panda_arm.xacro"/>
   <xacro:panda_arm arm_id="$(arg arm_id)" safety_distance="0.03"/>
@@ -27,3 +28,15 @@
     </xacro:if>
   </xacro:if>
+  <!-- RealSense camera -->
+  <xacro:if value="$(arg add_realsense)">
+    <!-- RealSense camera mount -->
+    <xacro:include filename="$(find mul_franka_description)/robots/panda_realsense_d435_camera_mount.xacro"/>
+    <xacro:panda_realsense_d435_camera_mount arm_id="$(arg arm_id)" connected_to="$(arg arm_id)_link8" xyz="0 0 0.0075" rpy="0 0 ${pi*3/4}"/>
+    <!-- RealSense camera -->
+    <!-- NOTE: The macro argument "name" has to match the parameter "camera_name" of the RealSense node. -->
+    <xacro:include filename="$(find realsense2_description)/urdf/_d435.urdf.xacro" />
+    <xacro:sensor_d435 name="camera" parent="$(arg arm_id)_realsense_mount_tip" use_nominal_extrinsics="false" add_plug="false" use_mesh="true">
+      <origin xyz="0.010025 0 -0.0115" />
+    </xacro:sensor_d435>
+  </xacro:if>
 </robot>

Commit message: make camera model configurable

File: mul_franka_description/robots/panda_arm.urdf.xacro (robot description, xacro)
@@ -6,5 +6,6 @@
   <xacro:arg name="use_fake_hardware" default="false"/>
   <xacro:arg name="fake_sensor_commands" default="false"/>
-  <xacro:arg name="add_realsense" default="false"/>
+  <xacro:arg name="camera" default=""/>
+  <xacro:property name="camera" value="$(arg camera)"/>
   <xacro:include filename="$(find franka_description)/robots/panda_arm.xacro"/>
   <xacro:panda_arm arm_id="$(arg arm_id)" safety_distance="0.03"/>
@@ -29,5 +30,5 @@
   </xacro:if>
   <!-- RealSense camera -->
-  <xacro:if value="$(arg add_realsense)">
+  <xacro:if value="${camera == 'realsense'}">
     <!-- RealSense camera mount -->
     <xacro:include filename="$(find mul_franka_description)/robots/panda_realsense_d435_camera_mount.xacro"/>

File: mul_franka_description/srdf/panda_arm.srdf.xacro (robot description, xacro)
@@ -3,5 +3,6 @@
   <xacro:arg name="arm_id" default="panda"/> <!-- Name of this panda -->
   <xacro:arg name="hand" default="true"/> <!-- Should a franka_gripper be mounted at the flange? (Currently does not work without it) -->
-  <xacro:arg name="add_realsense" default="false"/>
+  <xacro:arg name="camera" default=""/>
+  <xacro:property name="camera" value="$(arg camera)"/>
   <xacro:property name="arm_id" value="$(arg arm_id)"/>
   <xacro:include filename="$(find franka_moveit_config)/srdf/panda_arm.xacro"/>
@@ -13,5 +14,5 @@
     <xacro:panda_arm_hand arm_id="${arm_id}"/>
   </xacro:if>
-  <xacro:if value="$(arg add_realsense)">
+  <xacro:if value="${camera == 'realsense'}">
     <disable_collisions link1="${arm_id}_hand" link2="${arm_id}_realsense_link" reason="Adjacent"/>
     <disable_collisions link1="${arm_id}_hand" link2="${arm_id}_realsense_mount" reason="Adjacent"/>

Commit message: Femto Bolt mount and camera xacro

File: mul_franka_description/robots/panda_arm.urdf.xacro (robot description, xacro)
@@ -41,3 +41,14 @@
     </xacro:sensor_d435>
   </xacro:if>
+  <!-- Orbbec Femto camera -->
+  <xacro:if value="${camera == 'femto'}">
+    <!-- Femto Bolt camera mount -->
+    <xacro:include filename="$(find mul_franka_description)/robots/panda_femto_bolt_camera_mount.xacro"/>
+    <xacro:panda_femto_bolt_camera_mount arm_id="$(arg arm_id)" connected_to="$(arg arm_id)_link8" xyz="${sqrt(0.015**2/2)} -${sqrt(0.015**2/2)} 0.01915" rpy="${pi*-1/2} 0 ${pi*-3/4}"/>
+    <!-- Femto Bolt camera -->
+    <xacro:include filename="$(find orbbec_description)/urdf/femto_bolt.urdf.xacro" />
+    <xacro:femto_bolt prefix="camera" parent="$(arg arm_id)_femto_mount_tip" use_nominal_extrinsics="false">
+      <origin/>
+    </xacro:femto_bolt>
+  </xacro:if>
 </robot>

File: mul_franka_description/srdf/panda_arm.srdf.xacro (robot description, xacro)
@@ -22,3 +22,11 @@
     <disable_collisions link1="${arm_id}_realsense_link" link2="camera_link" reason="Adjacent"/>
   </xacro:if>
+  <xacro:if value="${camera == 'femto'}">
+    <disable_collisions link1="camera_base_link" link2="${arm_id}_hand" reason="Adjacent"/>
+    <disable_collisions link1="camera_base_link" link2="${arm_id}_link7" reason="Adjacent"/>
+    <disable_collisions link1="camera_base_link" link2="${arm_id}_link8" reason="Adjacent"/>
+    <disable_collisions link1="${arm_id}_femto_mount" link2="${arm_id}_hand" reason="Adjacent"/>
+    <disable_collisions link1="${arm_id}_femto_mount" link2="${arm_id}_link7" reason="Adjacent"/>
+    <disable_collisions link1="${arm_id}_femto_mount" link2="${arm_id}_link8" reason="Adjacent"/>
+  </xacro:if>
 </robot>
